Commit message: Ros archived

File: description/urdf/ads-dv.urdf.xacro (robot description, xacro)
@@ -6,9 +6,9 @@
     <!-- First we import all posible elements defined in the urdf.xacro files. All these elements are defined as macro:xacros -->
     <!-- Import Robotnik CAR base elements -->
-    <xacro:include filename="$(find eufs_description)/urdf/bases/ads-dv_base.urdf.xacro" />
+    <xacro:include filename="/mnt/c/Users/shuai/FSAI-PIONEERS/MIDDLESEX-UNI/description/urdf/bases/ads-dv_base.urdf.xacro" />
     <!-- Import Robotnik CAR wheels -->
-    <xacro:include filename="$(find eufs_description)/urdf/wheels/suspension_wheel.urdf.xacro" />
+    <xacro:include filename="/mnt/c/Users/shuai/FSAI-PIONEERS/MIDDLESEX-UNI/description/urdf/wheels/suspension_wheel.urdf.xacro" />
     <!-- Import all available sensors -->
-    <xacro:include filename="$(find eufs_description)/sensors/all_sensors.urdf.xacro" />
+    <xacro:include filename="/mnt/c/Users/shuai/FSAI-PIONEERS/MIDDLESEX-UNI/description/urdf/sensors/all_sensors.urdf.xacro" />
     <!-- ***************** -->
     <!-- Global parameters -->

File: description/urdf/bases/ads-dv_base.urdf.xacro (robot description, xacro)
@@ -1,5 +1,5 @@
 <?xml version="1.0"?>
 <robot name="eufs" xmlns:xacro="http://www.ros.org/wiki/xacro">
-  <xacro:include filename="$(find eufs_description)/urdf/bases/eufs_base.gazebo.xacro" />
+  <xacro:include filename="/mnt/c/Users/shuai/FSAI-PIONEERS/MIDDLESEX-UNI/description/urdf/bases/eufs_base.gazebo.xacro" />
   <xacro:macro name="eufs_base" params="name publish_bf hq">
   <!-- Robot mechanical and motor parameters -->
@@ -43,10 +43,10 @@
        <xacro:if value="${hq}">
        <geometry>
-	     <mesh filename="package://eufs_description/meshes/ads-dv.dae"/>
+	     <mesh filename="file:///mnt/c/Users/shuai/FSAI-PIONEERS/MIDDLESEX-UNI/description/meshes/ads-dv.dae"/>
        </geometry>
        </xacro:if>
        <xacro:unless value="${hq}">
        <geometry>
-	     <mesh filename="package://eufs_description/meshes/ads-dv.dae"/>
+	     <mesh filename="file:///mnt/c/Users/shuai/FSAI-PIONEERS/MIDDLESEX-UNI/description/meshes/ads-dv.dae"/>
        </geometry>
        </xacro:unless>
@@ -55,5 +55,5 @@
        <origin xyz="0 0 0" rpy="0 0 0 " />
        <geometry>
-         <mesh filename="package://eufs_description/meshes/ads-dv.dae"/>
+         <mesh filename="file:///mnt/c/Users/shuai/FSAI-PIONEERS/MIDDLESEX-UNI/description/meshes/ads-dv.dae"/>
        </geometry>
     </collision>

File: description/urdf/bases/eufs_base.urdf.xacro (robot description, xacro)
@@ -1,5 +1,5 @@
 <?xml version="1.0"?>
 <robot name="eufs" xmlns:xacro="http://www.ros.org/wiki/xacro">
-  <xacro:include filename="$(find eufs_description)/urdf/bases/eufs_base.gazebo.xacro" />
+  <xacro:include filename="/mnt/c/Users/shuai/FSAI-PIONEERS/MIDDLESEX-UNI/description/urdf/bases/eufs_base.gazebo.xacro" />
   <xacro:macro name="eufs_base" params="name publish_bf hq">
   <!-- Robot mechanical and motor parameters -->
@@ -43,10 +43,10 @@
        <xacro:if value="${hq}">
        <geometry>
-	     <mesh filename="package://eufs_description/meshes/chassis.dae"/>
+	     <mesh filename="file:///mnt/c/Users/shuai/FSAI-PIONEERS/MIDDLESEX-UNI/description/meshes/chassis.dae"/>
        </geometry>
        </xacro:if>
        <xacro:unless value="${hq}">
        <geometry>
-	     <mesh filename="package://eufs_description/meshes/chassis.dae"/>
+	     <mesh filename="file:///mnt/c/Users/shuai/FSAI-PIONEERS/MIDDLESEX-UNI/description/meshes/chassis.dae"/>
        </geometry>
        </xacro:unless>
@@ -55,5 +55,5 @@
        <origin xyz="0 0 0" rpy="0 0 0 " />
        <geometry>
-         <mesh filename="package://eufs_description/meshes/chassis_collision.dae"/>
+         <mesh filename="file:///mnt/c/Users/shuai/FSAI-PIONEERS/MIDDLESEX-UNI/description/meshes/chassis_collision.dae"/>
        </geometry>
     </collision>
